File: Match_Maker_NPN_PNP/Core_Circuit.kicad_sch (KiCad schematic)
At the start: 0 parts

Commit message: Created schematic
Parts:
- added Q1, Q2: BC548, Package_TO_SOT_THT:TO-92_Inline, symbol Transistor_BJT:BC548
- added Q3, Q4: BC558, Package_TO_SOT_THT:TO-92_Inline, symbol Transistor_BJT:BC558
- added R1, R2, R3, R4, R5, R6: 10K, Resistor_THT:R_Axial_DIN0207_L6.3mm_D2.5mm_P7.62mm_Horizontal, symbol Device:R_US
- added R7, R8: 68k, Resistor_THT:R_Axial_DIN0207_L6.3mm_D2.5mm_P7.62mm_Horizontal, symbol Device:R_US
- added TP1, TP3: +, symbol Connector:TestPoint
- added TP2, TP4: -, symbol Connector:TestPoint
- added U1: TL072, symbol Amplifier_Operational:TL072
Connections:
- new net: Q1.3 (E), R5.1, TP2.1
- new net: R3.1, R4.1, U1.5 (+)
- new net: Q3.3 (E), R8.2, U1.6 (-)
- new net: Q3.2 (B), U1.7
- new net: Q3.1 (C), R6.1
- new net: Q2.1 (C), R5.2
- new net: R1.1, R2.1, U1.3 (+)
- new net: Q4.3 (E), R6.2, TP3.1
- new net: Q2.2 (B), U1.1
- new net: Q2.3 (E), R7.1, U1.2 (-)
- new net +12V: Q1.1 (C), R4.2, R8.1
- new net -12V: Q4.1 (C), R2.2, R7.2
- new net GND: Q1.2 (B), Q4.2 (B), R1.2, R3.2, TP1.1, TP4.1
