File: Match_Maker_NPN_PNP/Power.kicad_sch (KiCad schematic)
At the start: 14 parts, among them J0 Conn_01x01, J100 IDC_02x08, J101 IDC_02x05

Commit message: Created schematic
Parts:
- removed C3: 47uF, Capacitor_THT:CP_Radial_D4.0mm_P1.50mm, symbol Device:C_Polarized
- removed C6: 100nF, Capacitor_THT:C_Disc_D4.3mm_W1.9mm_P5.00mm, symbol Device:C
- removed D1, D3: SB140+, Diode_THT:D_DO-41_SOD81_P10.16mm_Horizontal, symbol SynthStuff:Power_Bus_Schotty_+
- removed D2: SB140-, Diode_THT:D_DO-41_SOD81_P10.16mm_Horizontal, symbol SynthStuff:Power_Bus_Schotty_-
- removed J100: IDC_02x08, SynthStuff:IDC-Header_2x08_P2.54mm_Vertical_Eurorack, symbol SynthStuff:Eurorack_Power_Connector_16Pin
- added U1: TL072, symbol Amplifier_Operational:TL072
- renumbered J101 to J100
Connections:
- net +12V: now also U1.8 (V+)
- net -12V: now also U1.4 (V-)
Other:
- note removed: "Delete what's not needed!"
